File: gbcart.kicad_pcb (KiCad board)
At the start: 2 copper layers, 51.4 x 61 mm, 40 parts, among them J1 Conn_01x32, J2 USB_B_Micro, J3 Micro_SD_Card, J4 Conn_01x06_Male, J5 Conn_01x06_Male, Q1 BC847, SW1 SW_Push, U1 ESP32-S3-MINI-1, U2 74HC138, U3 74HCT1G125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

Commit message: Generate production files
Other:
- board text added: "v2.0"
- board text removed: "DEV"
Changed lines of the file:
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@@
       (drillshape 0)
       (scaleselection 1)
-      (outputdirectory "gerbers/")
+      (outputdirectory "gbusbcart/gerbers/")
     )
   )
@@
   (gr_line locked (start 149.525 62.595) (end 145.525 62.595) (layer "Edge.Cuts") (width 0.15))
   (gr_line locked (start 99.225 112.395) (end 98.125 112.395) (layer "Edge.Cuts") (width 0.15))
-  (gr_text "DEV" (at 128.27 89.154) (layer "B.Cu")
+  (gr_text "v2.0" (at 128.27 89.154) (layer "B.Cu")
     (effects (font (size 1.5 1.5) (thickness 0.3)) (justify mirror))
   )
