File: gbcart_sim.kicad_sch (KiCad schematic)
At the start: 27 parts, among them J1 Micro_SD_Card, J2 Conn_02x17_Odd_Even, J3 Conn_01x32, Q1 BC847, SW1 SW_Push, U1 ESP32-S3-DevKitC, U2 74lxc125, U3 74HC138, U4 74HCT1G125, U5 74HC259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

Commit message: Fix board
Parts:
- gave numbers to parts that had none: 1
Changed lines of the file:
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@@
   (symbol (lib_id "power:+5V") (at 106.68 114.3 0) (unit 1)
     (in_bom yes) (on_board yes) (fields_autoplaced)
-    (property "Reference" "#PWR?" (id 0) (at 106.68 118.11 0)
+    (property "Reference" "#PWR0107" (id 0) (at 106.68 118.11 0)
       (effects (font (size 1.27 1.27)) hide)
     )
@@
   (symbol (lib_id "power:GND") (at 105.41 110.49 180) (unit 1)
     (in_bom yes) (on_board yes) (fields_autoplaced)
-    (property "Reference" "#PWR?" (id 0) (at 105.41 104.14 0)
+    (property "Reference" "#PWR0105" (id 0) (at 105.41 104.14 0)
       (effects (font (size 1.27 1.27)) hide)
     )
@@
   (symbol (lib_id "power:GND") (at 106.68 116.84 0) (unit 1)
     (in_bom yes) (on_board yes) (fields_autoplaced)
-    (property "Reference" "#PWR?" (id 0) (at 106.68 123.19 0)
+    (property "Reference" "#PWR0106" (id 0) (at 106.68 123.19 0)
       (effects (font (size 1.27 1.27)) hide)
     )
@@
   (symbol (lib_id "74xGxx:74AHC1G125") (at 105.41 115.57 0) (unit 1)
     (in_bom yes) (on_board yes) (fields_autoplaced)
-    (property "Reference" "U?" (id 0) (at 104.775 120.65 0))
+    (property "Reference" "U7" (id 0) (at 104.775 120.65 0))
     (property "Value" "74HCT1G125" (id 1) (at 104.775 123.19 0))
     (property "Footprint" "Package_TO_SOT_SMD:SOT-353_SC-70-5_Handsoldering" (id 2) (at 105.41 115.57 0)
@@
       (reference "#PWR0104") (unit 1) (value "+3.3V") (footprint "")
     )
+    (path "/523411b2-3603-4b3e-b6f3-7fd68a08189a"
+      (reference "#PWR0105") (unit 1) (value "GND") (footprint "")
+    )
+    (path "/dfd72bdc-4a88-46a1-a956-4f5f7f5612c0"
+      (reference "#PWR0106") (unit 1) (value "GND") (footprint "")
+    )
     (path "/4322f36d-0131-46df-9889-eb45983e57c3"
-      (reference "#PWR?") (unit 1) (value "+5V") (footprint "")
-    )
-    (path "/523411b2-3603-4b3e-b6f3-7fd68a08189a"
-      (reference "#PWR?") (unit 1) (value "GND") (footprint "")
-    )
-    (path "/dfd72bdc-4a88-46a1-a956-4f5f7f5612c0"
-      (reference "#PWR?") (unit 1) (value "GND") (footprint "")
+      (reference "#PWR0107") (unit 1) (value "+5V") (footprint "")
     )
     (path "/49ce2515-fd5a-40e0-9860-0e59365ec9c8"
@@
     )
     (path "/fc9177a7-bc41-4270-bf1d-f64afb558963"
-      (reference "U?") (unit 1) (value "74HCT1G125") (footprint "Package_TO_SOT_SMD:SOT-353_SC-70-5_Handsoldering")
-    )
-  )
+      (reference "U7") (unit 1) (value "74HCT1G125") (footprint "Package_TO_SOT_SMD:SOT-353_SC-70-5_Handsoldering")
+    )
+  )
